Commit message: US_10825: urdf modifications

File: Software/ros2_ws/src/atv/urdf/snower.urdf (robot description, URDF)
Before this commit: robot robot_description, 3 links, 2 joints
Links:
- removed link zed_camera_link
- added link snower/zed2_camera_link
Joints:
- joint base_to_zed2: child zed_camera_link -> snower/zed2_camera_link

Commit message: US_10825: udrf modification

File: Software/ros2_ws/src/atv/urdf/snower.urdf (robot description, URDF)
Before this commit: robot robot_description, 3 links, 2 joints
Joints:
- joint base_to_os_sensor: origin xyz=0 0 0.5 rpy=0 0 0 -> xyz=0 0 0 rpy=0 0 0
- joint base_to_zed2: origin xyz=0.75 0 0.5 rpy=0 0 0 -> xyz=0 0 0 rpy=0 0 0

Commit message: US_10825: odom modifications

File: Software/ros2_ws/src/atv/urdf/snower.urdf (robot description, URDF)
Before this commit: robot robot_description, 3 links, 2 joints
Links:
- added link snower/gnss_link
Joints:
- added joint base_gnss: type fixed, parent base_link, child snower/gnss_link, origin xyz=0 0 0 rpy=0 0 0
