Commit message: US_10825: added the collisions for xacro files

File: Software/ros2_ws/src/atv/urdf/ouster_lidar.xacro (robot description, xacro)
@@ -21,4 +21,18 @@
         <material name="orange"/>
       </visual>
+      <collision>
+      <origin xyz="0 0 0"/>
+         <geometry>
+           <cylinder length="0.074" radius="0.04" />
+         </geometry>
+         <material name="orange"/>
+      </collision>
+      <collision>
+        <origin xyz="0 0 -0.045"/>
+        <geometry>
+          <box size="0.112 0.112 0.016" />
+        </geometry>
+        <material name="orange"/>
+      </collision>
   </link>
 </robot>

File: Software/ros2_ws/src/atv/urdf/snower_core.xacro (robot description, xacro)
@@ -43,4 +43,18 @@
             <material name="white"/>
         </visual>
+        <collision>
+            <origin xyz="0 0 0"/>
+            <geometry>
+                <box size="0.92 0.5 0.32"/>
+            </geometry>
+            <material name="white"/>
+        </collision>
+        <collision>
+            <origin xyz="0.3 0 0.31"/>
+            <geometry>
+                <cylinder radius="0.05" length="0.3"/>
+            </geometry>
+            <material name="white"/>
+        </collision>
     </link>
     <!-- LEFT BACK WHEEL LINK -->
@@ -58,4 +72,10 @@
             <material name="black"/>
         </visual>
+        <collision>
+            <geometry>
+                <cylinder radius="0.15" length="0.30"/>
+            </geometry>
+            <material name="black"/>
+        </collision>
     </link>
     <!-- RIGHT BACK WHEEL LINK -->
@@ -73,4 +93,10 @@
             <material name="black"/>
         </visual>
+        <collision>
+            <geometry>
+                <cylinder radius="0.15" length="0.30"/>
+            </geometry>
+            <material name="black"/>
+        </collision>
     </link>
     <!-- LEFT FRONT WHEEL LINK -->
@@ -88,4 +114,10 @@
             <material name="black"/>
         </visual>
+        <collision>
+            <geometry>
+                <cylinder radius="0.15" length="0.30"/>
+            </geometry>
+            <material name="black"/>
+        </collision>
     </link>
     <!-- RIGHT FRONT WHEEL LINK -->
@@ -103,4 +135,10 @@
             <material name="black"/>
         </visual>
+        <collision>
+            <geometry>
+                <cylinder radius="0.15" length="0.30"/>
+            </geometry>
+            <material name="black"/>
+        </collision>
     </link>
 </robot>

File: Software/ros2_ws/src/atv/urdf/zed2_camara.xacro (robot description, xacro)
@@ -14,4 +14,11 @@
           <material name="orange"/>
       </visual>
+      <collision>
+          <origin xyz="0 0 0"/>
+          <geometry>
+              <box size="0.030 0.175 0.033"/>
+          </geometry>
+          <material name="orange"/>
+      </collision>
   </link>
 </robot>

File: Software/ros2_ws/src/atv/urdf/zedf9p_gnss.xacro (robot description, xacro)
@@ -14,4 +14,11 @@
           <material name="orange"/>
       </visual>
+      <collision>
+          <origin xyz="0 0 0"/>
+          <geometry>
+              <box size="0.063 0.067 0.026"/>
+          </geometry>
+          <material name="orange"/>
+      </collision>
   </link>
 </robot>

Commit message: US_10825: formatted xacro files

File: Software/ros2_ws/src/atv/urdf/ouster_lidar.xacro (robot description, xacro)
@@ -1,38 +1,38 @@
 <?xml version="1.0"?>
-<robot xmlns:xacro="http://www.ros.org/wiki/xacro" >
+<robot xmlns:xacro="http://www.ros.org/wiki/xacro">
   <joint name="base_to_lidar" type="fixed">
-      <parent link="base_link"/>
-      <child link="os_sensor"/>
-      <origin xyz="0.3 0 0.753"/>
+    <parent link="base_link" />
+    <child link="os_sensor" />
+    <origin xyz="0.3 0 0.753" />
   </joint>
   <link name="os_sensor">
-      <visual>
-      <origin xyz="0 0 0"/>
-         <geometry>
-           <cylinder length="0.074" radius="0.04" />
-         </geometry>
-         <material name="orange"/>
-      </visual>
-      <visual>
-        <origin xyz="0 0 -0.045"/>
-        <geometry>
-          <box size="0.112 0.112 0.016" />
-        </geometry>
-        <material name="orange"/>
-      </visual>
-      <collision>
-      <origin xyz="0 0 0"/>
-         <geometry>
-           <cylinder length="0.074" radius="0.04" />
-         </geometry>
-         <material name="orange"/>
-      </collision>
-      <collision>
-        <origin xyz="0 0 -0.045"/>
-        <geometry>
-          <box size="0.112 0.112 0.016" />
-        </geometry>
-        <material name="orange"/>
-      </collision>
+    <visual>
+      <origin xyz="0 0 0" />
+      <geometry>
+        <cylinder length="0.074" radius="0.04" />
+      </geometry>
+      <material name="orange" />
+    </visual>
+    <visual>
+      <origin xyz="0 0 -0.045" />
+      <geometry>
+        <box size="0.112 0.112 0.016" />
+      </geometry>
+      <material name="orange" />
+    </visual>
+    <collision>
+      <origin xyz="0 0 0" />
+      <geometry>
+        <cylinder length="0.074" radius="0.04" />
+      </geometry>
+      <material name="orange" />
+    </collision>
+    <collision>
+      <origin xyz="0 0 -0.045" />
+      <geometry>
+        <box size="0.112 0.112 0.016" />
+      </geometry>
+      <material name="orange" />
+    </collision>
   </link>
 </robot>

File: Software/ros2_ws/src/atv/urdf/snower.urdf.xacro (robot description, xacro)
@@ -1,4 +1,4 @@
 <?xml version="1.0"?>
-<robot xmlns:xacro="http://www.ros.org/wiki/xacro"  name="snower">
+<robot xmlns:xacro="http://www.ros.org/wiki/xacro" name="snower">
     <xacro:include filename="snower_core.xacro" />
     <xacro:include filename="zed2_camara.xacro" />

File: Software/ros2_ws/src/atv/urdf/snower_core.xacro (robot description, xacro)
@@ -1,22 +1,22 @@
 <?xml version="1.0"?>
-<robot xmlns:xacro="http://www.ros.org/wiki/xacro" >
-    <xacro:include filename="inertial_macros.xacro"/>
+<robot xmlns:xacro="http://www.ros.org/wiki/xacro">
+    <xacro:include filename="inertial_macros.xacro" />
     <material name="white">
         <color rgba="1 1 1 0.9" />
     </material>
     <material name="orange">
-        <color rgba="1 0.3 0.1 1"/>
+        <color rgba="1 0.3 0.1 1" />
     </material>
     <material name="blue">
-        <color rgba="0.2 0.2 1 1"/>
+        <color rgba="0.2 0.2 1 1" />
     </material>
     <material name="red">
-        <color rgba="1 0 0 1"/>
+        <color rgba="1 0 0 1" />
     </material>
     <material name="green">
-        <color rgba="0 1 0 1"/>
+        <color rgba="0 1 0 1" />
     </material>
     <material name="black">
-        <color rgba="0.15 0.15 0.15 1"/>
+        <color rgba="0.15 0.15 0.15 1" />
     </material>
     <!-- BASE LINK -->
@@ -24,120 +24,120 @@
     <!-- CHASSIS LINK -->
     <joint name="chassis_joint" type="fixed">
-        <parent link="base_link"/>
-        <child link="chassis_link"/>
-        <origin xyz="0 0 0.24"/>
+        <parent link="base_link" />
+        <child link="chassis_link" />
+        <origin xyz="0 0 0.24" />
     </joint>
     <link name="chassis_link">
         <visual>
-            <origin xyz="0 0 0"/>
+            <origin xyz="0 0 0" />
             <geometry>
-                <box size="0.92 0.5 0.32"/>
+                <box size="0.92 0.5 0.32" />
             </geometry>
-            <material name="white"/>
+            <material name="white" />
         </visual>
         <visual>
-            <origin xyz="0.3 0 0.31"/>
+            <origin xyz="0.3 0 0.31" />
             <geometry>
-                <cylinder radius="0.05" length="0.3"/>
+                <cylinder radius="0.05" length="0.3" />
             </geometry>
-            <material name="white"/>
+            <material name="white" />
         </visual>
         <collision>
-            <origin xyz="0 0 0"/>
+            <origin xyz="0 0 0" />
             <geometry>
-                <box size="0.92 0.5 0.32"/>
+                <box size="0.92 0.5 0.32" />
             </geometry>
-            <material name="white"/>
+            <material name="white" />
         </collision>
         <collision>
-            <origin xyz="0.3 0 0.31"/>
+            <origin xyz="0.3 0 0.31" />
             <geometry>
-                <cylinder radius="0.05" length="0.3"/>
+                <cylinder radius="0.05" length="0.3" />
             </geometry>
-            <material name="white"/>
+            <material name="white" />
         </collision>
     </link>
     <!-- LEFT BACK WHEEL LINK -->
     <joint name="left_back_wheel_joint" type="fixed">
-        <parent link="base_link"/>
-        <child link="left_back_wheel_link"/>
+        <parent link="base_link" />
+        <child link="left_back_wheel_link" />
         <origin xyz="-0.26 0.41 0.15" rpy="-${pi/2} 0 0" />
-        <axis xyz="0 0 1"/>
+        <axis xyz="0 0 1" />
     </joint>
     <link name="left_back_wheel_link">
         <visual>
             <geometry>
-                <cylinder radius="0.15" length="0.30"/>
+                <cylinder radius="0.15" length="0.30" />
             </geometry>
-            <material name="black"/>
+            <material name="black" />
         </visual>
         <collision>
             <geometry>
-                <cylinder radius="0.15" length="0.30"/>
+                <cylinder radius="0.15" length="0.30" />
             </geometry>
-            <material name="black"/>
+            <material name="black" />
         </collision>
     </link>
     <!-- RIGHT BACK WHEEL LINK -->
     <joint name="right_back_wheel_joint" type="fixed">
-        <parent link="base_link"/>
-        <child link="right_back_wheel_link"/>
+        <parent link="base_link" />
+        <child link="right_back_wheel_link" />
         <origin xyz="-0.26 -0.41 0.15" rpy="${pi/2} 0 0" />
-        <axis xyz="0 0 -1"/>
+        <axis xyz="0 0 -1" />
     </joint>
     <link name="right_back_wheel_link">
         <visual>
             <geometry>
-                <cylinder radius="0.15" length="0.30"/>
+                <cylinder radius="0.15" length="0.30" />
             </geometry>
-            <material name="black"/>
+            <material name="black" />
         </visual>
         <collision>
             <geometry>
-                <cylinder radius="0.15" length="0.30"/>
+                <cylinder radius="0.15" length="0.30" />
             </geometry>
-            <material name="black"/>
+            <material name="black" />
         </collision>
     </link>
     <!-- LEFT FRONT WHEEL LINK -->
     <joint name="left_front_wheel_joint" type="fixed">
-        <parent link="base_link"/>
-        <child link="left_front_wheel_link"/>
+        <parent link="base_link" />
+        <child link="left_front_wheel_link" />
         <origin xyz="0.26 0.41 0.15" rpy="-${pi/2} 0 0" />
-        <axis xyz="0 0 1"/>
+        <axis xyz="0 0 1" />
     </joint>
     <link name="left_front_wheel_link">
         <visual>
             <geometry>
-                <cylinder radius="0.15" length="0.30"/>
+                <cylinder radius="0.15" length="0.30" />
             </geometry>
-            <material name="black"/>
+            <material name="black" />
         </visual>
         <collision>
             <geometry>
-                <cylinder radius="0.15" length="0.30"/>
+                <cylinder radius="0.15" length="0.30" />
             </geometry>
-            <material name="black"/>
+            <material name="black" />
         </collision>
     </link>
     <!-- RIGHT FRONT WHEEL LINK -->
     <joint name="right_front_wheel_joint" type="fixed">
-        <parent link="base_link"/>
-        <child link="right_front_wheel_link"/>
+        <parent link="base_link" />
+        <child link="right_front_wheel_link" />
         <origin xyz="0.26 -0.41 0.15" rpy="${pi/2} 0 0" />
-        <axis xyz="0 0 -1"/>
+        <axis xyz="0 0 -1" />
     </joint>
     <link name="right_front_wheel_link">
         <visual>
             <geometry>
-                <cylinder radius="0.15" length="0.30"/>
+                <cylinder radius="0.15" length="0.30" />
             </geometry>
-            <material name="black"/>
+            <material name="black" />
         </visual>
         <collision>
             <geometry>
-                <cylinder radius="0.15" length="0.30"/>
+                <cylinder radius="0.15" length="0.30" />
             </geometry>
-            <material name="black"/>
+            <material name="black" />
         </collision>
     </link>

File: Software/ros2_ws/src/atv/urdf/zed2_camara.xacro (robot description, xacro)
@@ -1,24 +1,24 @@
 <?xml version="1.0"?>
-<robot xmlns:xacro="http://www.ros.org/wiki/xacro" >
-  <joint name="base_to_zed2" type="fixed">
-      <parent link="base_link"/>
-      <child link="zed2_camera_link"/>
-      <origin xyz="0.445 0 0.4165"/>
-  </joint>
-  <link name="zed2_camera_link">
-      <visual>
-          <origin xyz="0 0 0"/>
-          <geometry>
-              <box size="0.030 0.175 0.033"/>
-          </geometry>
-          <material name="orange"/>
-      </visual>
-      <collision>
-          <origin xyz="0 0 0"/>
-          <geometry>
-              <box size="0.030 0.175 0.033"/>
-          </geometry>
-          <material name="orange"/>
-      </collision>
-  </link>
+<robot xmlns:xacro="http://www.ros.org/wiki/xacro">
+    <joint name="base_to_zed2" type="fixed">
+        <parent link="base_link" />
+        <child link="zed2_camera_link" />
+        <origin xyz="0.445 0 0.4165" />
+    </joint>
+    <link name="zed2_camera_link">
+        <visual>
+            <origin xyz="0 0 0" />
+            <geometry>
+                <box size="0.030 0.175 0.033" />
+            </geometry>
+            <material name="orange" />
+        </visual>
+        <collision>
+            <origin xyz="0 0 0" />
+            <geometry>
+                <box size="0.030 0.175 0.033" />
+            </geometry>
+            <material name="orange" />
+        </collision>
+    </link>
 </robot>

File: Software/ros2_ws/src/atv/urdf/zedf9p_gnss.xacro (robot description, xacro)
@@ -1,24 +1,24 @@
 <?xml version="1.0"?>
-<robot xmlns:xacro="http://www.ros.org/wiki/xacro" >
-  <joint name="base_to_gnss" type="fixed">
-      <parent link="base_link"/>
-      <child link="gnss_link"/>
-      <origin xyz="-0.41 0.2 0.413"/>
-  </joint>
-  <link name="gnss_link">
-      <visual>
-          <origin xyz="0 0 0"/>
-          <geometry>
-              <box size="0.063 0.067 0.026"/>
-          </geometry>
-          <material name="orange"/>
-      </visual>
-      <collision>
-          <origin xyz="0 0 0"/>
-          <geometry>
-              <box size="0.063 0.067 0.026"/>
-          </geometry>
-          <material name="orange"/>
-      </collision>
-  </link>
+<robot xmlns:xacro="http://www.ros.org/wiki/xacro">
+    <joint name="base_to_gnss" type="fixed">
+        <parent link="base_link" />
+        <child link="gnss_link" />
+        <origin xyz="-0.41 0.2 0.413" />
+    </joint>
+    <link name="gnss_link">
+        <visual>
+            <origin xyz="0 0 0" />
+            <geometry>
+                <box size="0.063 0.067 0.026" />
+            </geometry>
+            <material name="orange" />
+        </visual>
+        <collision>
+            <origin xyz="0 0 0" />
+            <geometry>
+                <box size="0.063 0.067 0.026" />
+            </geometry>
+            <material name="orange" />
+        </collision>
+    </link>
 </robot>
