Commit message: US_10825: zed2 camara link

File: Software/ros2_ws/src/atv/urdf/zed2_camara.xacro (robot description, xacro)
@@ -3,8 +3,8 @@
     <joint name="base_to_zed2" type="fixed">
         <parent link="base_link" />
-        <child link="zed2_camera_link" />
+        <child link="zed_camera_link" />
         <origin xyz="0.445 0 0.4165" />
     </joint>
-    <link name="zed2_camera_link">
+    <link name="zed_camera_link">
         <visual>
             <origin xyz="0 0 0" />
