Commit message: US_11756: base_footprint

File: Software/ros2_ws/src/atv/urdf/snower_core.xacro (robot description, xacro)
@@ -19,6 +19,14 @@
         <color rgba="0.15 0.15 0.15 1" />
     </material>
-    <!-- BASE LINK -->
-    <link name="base_link"></link>
+    <link name="base_footprint">
+    </link>
+    <!-- BASE_FOOTPRINT LINK -->
+    <joint name="base_footprint_joint" type="fixed">
+        <parent link="base_footprint"/>
+        <child link="base_link"/>
+        <origin xyz="0 0 0" rpy="0 0 0"/>
+    </joint>
+    <link name="base_link">
+    </link>
     <!-- CHASSIS LINK -->
     <joint name="chassis_joint" type="fixed">
