File: Hardware/universal_power_distribution_PCB/universal_power_distribution_PCB.kicad_sch (KiCad schematic)
At the start: 0 parts

Commit message: Updated universal PCB
Other:
- company: (none) -> Lapin AMK
- title: (none) -> Power distribution pcb

Commit message: Restructured pcb
Other:
- added sheet connectors (connectors.kicad_sch)
- added sheet current_sensing (current_sensing.kicad_sch)
Changed lines of the file:
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@@
+		)
+	)
+	(sheet
+		(at 33.02 63.5)
+		(size 43.18 13.97)
+		(fields_autoplaced yes)
+		(stroke
+			(width 0.1524)
+			(type solid)
+		)
+		(fill
+			(color 0 0 0 0.0000)
+		)
+		(property "Sheetname" "current_sensing"
+			(at 33.02 62.7884 0)
+			(effects
+				(font
+					(size 1.27 1.27)
+				)
+				(justify left bottom)
+			)
+		)
+		(property "Sheetfile" "current_sensing.kicad_sch"
+			(at 33.02 78.0546 0)
+			(effects
+				(font
+					(size 1.27 1.27)
+				)
+				(justify left top)
+				(hide yes)
+			)
+		)
+		(instances
+			(project "universal_power_distribution_PCB"
+				(path "/7b61ee4e-2c0c-4866-8343-5ee759f84d1a"
+					(page "3")
+				)
+			)
+		)
+	)
+	(sheet
+		(at 33.02 87.63)
+		(size 43.18 12.7)
+		(fields_autoplaced yes)
+		(stroke
+			(width 0.1524)
+			(type solid)
+		)
+		(fill
+			(color 0 0 0 0.0000)
+		)
+		(property "Sheetname" "connectors"
+			(at 33.02 86.9184 0)
+			(effects
+				(font
+					(size 1.27 1.27)
+				)
+				(justify left bottom)
+			)
+		)
+		(property "Sheetfile" "connectors.kicad_sch"
+			(at 33.02 100.9146 0)
+			(effects
+				(font
+					(size 1.27 1.27)
+				)
+				(justify left top)
+			)
+		)
+		(instances
+			(project "universal_power_distribution_PCB"
+				(path "/7b61ee4e-2c0c-4866-8343-5ee759f84d1a"
+					(page "4")
+				)
+			)
 		)
 	)
