File: Hardware/UPD_PCB/Block Diagram.kicad_sch (KiCad schematic)
At the start: 0 parts

Commit message: Updated schematic (before INA219 integration)
Other:
- note removed: "+??V"
- note removed: "+A3V3"
