File: Hardware/UPD_PCB/Block Diagram.kicad_sch (KiCad schematic)
At the start: 0 parts

Commit message: Finalized Schematic
Other:
- title: Block Diagram -> Sheet Title A
Changed lines of the file:
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@@
 	(paper "A3")
 	(title_block
-		(title "Block Diagram")
+		(title "Sheet Title A")
 		(date "Last Modified Date")
 		(rev "${REVISION}")

Commit message: Updated pcb
Changed lines of the file:
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@@
 	)
 	(rectangle
-		(start 330.2 236.22)
-		(end 401.32 236.982)
+		(start 328.93 233.68)
+		(end 400.05 234.442)
 		(stroke
 			(width 0)
@@
 	)
 	(rectangle
-		(start 330.2 179.07)
-		(end 401.32 179.832)
+		(start 328.93 170.18)
+		(end 400.05 170.942)
 		(stroke
 			(width 0)
@@
 	(text_box "Out 2\n"
 		(exclude_from_sim no)
-		(at 331.47 198.12 0)
+		(at 330.2 189.23 0)
 		(size 41.91 7.62)
 		(stroke
@@
 	(text_box "Out 1"
 		(exclude_from_sim no)
-		(at 331.47 190.5 0)
+		(at 330.2 181.61 0)
 		(size 43.18 7.62)
 		(stroke
@@
 	(text_box "16V (2A)"
 		(exclude_from_sim no)
-		(at 377.19 213.36 0)
+		(at 375.92 204.47 0)
 		(size 27.94 7.62)
 		(stroke
@@
 	(text_box "Input voltage:"
 		(exclude_from_sim no)
-		(at 330.2 182.88 0)
+		(at 328.93 173.99 0)
 		(size 41.91 7.62)
 		(stroke
@@
 	(text_box "19V (2A)"
 		(exclude_from_sim no)
-		(at 377.19 205.74 0)
+		(at 375.92 196.85 0)
 		(size 29.21 7.62)
 		(stroke
@@
 	(text_box "36 V (25A)"
 		(exclude_from_sim no)
-		(at 377.19 190.5 0)
+		(at 375.92 181.61 0)
 		(size 27.94 7.62)
 		(stroke
@@
 		)
 	)
-	(text_box "5V (2A)"
-		(exclude_from_sim no)
-		(at 377.19 228.6 0)
+	(text_box "12V (2A)"
+		(exclude_from_sim no)
+		(at 375.92 219.71 0)
 		(size 29.21 7.62)
 		(stroke
@@
 				(face "Times New Roman")
 				(size 3.048 3.048)
+				(color 0 0 0 1)
+			)
+			(justify left top)
+		)
+	)
+	(text_box "Out 7"
+		(exclude_from_sim no)
+		(at 330.2 227.33 0)
+		(size 44.45 7.62)
+		(stroke
+			(width -0.0001)
+			(type default)
+		)
+		(fill
+			(type none)
+		)
+		(effects
+			(font
+				(face "Times New Roman")
+				(size 3.048 3.048)
+				(thickness 0.4572)
+				(bold yes)
 				(color 0 0 0 1)
 			)
@@
 	(text_box "Out 4"
 		(exclude_from_sim no)
-		(at 331.47 213.36 0)
+		(at 330.2 204.47 0)
 		(size 43.18 7.62)
 		(stroke
@@
 	(text_box "Target specifications:"
 		(exclude_from_sim no)
-		(at 327.66 171.45 0)
+		(at 326.39 162.56 0)
 		(size 73.66 7.62)
 		(stroke
@@
 	(text_box "24V (2A)"
 		(exclude_from_sim no)
-		(at 377.19 198.12 0)
+		(at 375.92 189.23 0)
 		(size 27.94 7.62)
 		(stroke
@@
 	(text_box "Out 6"
 		(exclude_from_sim no)
-		(at 331.47 228.6 0)
+		(at 330.2 219.71 0)
 		(size 44.45 7.62)
 		(stroke
@@
 	(text_box "42 - 36 V"
 		(exclude_from_sim no)
-		(at 375.92 182.88 0)
+		(at 374.65 173.99 0)
 		(size 24.13 7.62)
 		(stroke
@@
 	(text_box "12V (2A)"
 		(exclude_from_sim no)
-		(at 377.19 220.98 0)
+		(at 375.92 212.09 0)
 		(size 30.48 7.62)
 		(stroke
@@
 		)
 	)
+	(text_box "5V (2A)"
+		(exclude_from_sim no)
+		(at 375.92 227.33 0)
+		(size 29.21 7.62)
+		(stroke
+			(width -0.0001)
+			(type default)
+		)
+		(fill
+			(type none)
+		)
+		(effects
+			(font
+				(face "Times New Roman")
+				(size 3.048 3.048)
+				(color 0 0 0 1)
+			)
+			(justify left top)
+		)
+	)
 	(text_box "Out 5"
 		(exclude_from_sim no)
-		(at 331.47 220.98 0)
+		(at 330.2 212.09 0)
 		(size 41.91 7.62)
 		(stroke
@@
 	(text_box "Out 3"
 		(exclude_from_sim no)
-		(at 331.47 205.74 0)
+		(at 330.2 196.85 0)
 		(size 44.45 7.62)
 		(stroke
