File: Hardware/UPD_PCB/Power - Sequencing.kicad_sch (KiCad schematic)
At the start: 0 parts

Commit message: Finalized Schematic
Other:
- title: Power - Sequencing -> Sheet Title A
Changed lines of the file:
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@@
 	(paper "A4")
 	(title_block
-		(title "Power - Sequencing")
+		(title "Sheet Title A")
 		(date "Last Modified Date")
 		(rev "${REVISION}")
