File: Hardware/UPD_PCB/Power - Sequencing.kicad_sch (KiCad schematic)
At the start: 0 parts

Commit message: Finalized version V1.0
Other:
- note added: "0 to 5 volt uses a 4ms Soft start Other voltages are unknown untill physically tested"
