File: Hardware/UPD_PCB/UPD_PCB.kicad_pcb (KiCad board)
At the start: 6 copper layers, 0 parts

Commit message: Finalized Schematic
Parts:
- added C1: 2.2µF, Capacitor_SMD:C_0603_1608Metric_Pad1.08x0.95mm_HandSolder, F.Cu at (369.4, 37.2)
- added C10: 2.2µF, Capacitor_SMD:C_0603_1608Metric_Pad1.08x0.95mm_HandSolder, F.Cu at (369.4, 52.2)
- added C11: 2.2µF, Capacitor_SMD:C_0603_1608Metric_Pad1.08x0.95mm_HandSolder, F.Cu at (369.4, 54.7)
- added C12: DNP, Capacitor_SMD:C_0603_1608Metric_Pad1.08x0.95mm_HandSolder, F.Cu at (373.8, 37.2)
- added C13: DNP, Capacitor_SMD:C_0603_1608Metric_Pad1.08x0.95mm_HandSolder, F.Cu at (373.8, 39.7)
- added C14: 0.1µF, Capacitor_SMD:C_0603_1608Metric_Pad1.08x0.95mm_HandSolder, F.Cu at (373.8, 42.2)
- added C15: 0.1µF, Capacitor_SMD:C_0603_1608Metric_Pad1.08x0.95mm_HandSolder, F.Cu at (373.8, 44.7)
- added C16: 22µF, Capacitor_SMD:CP_Elec_6.3x5.8, F.Cu at (377.6, 15.5)
- added C17: 10µF, Capacitor_SMD:CP_Elec_6.3x5.8, F.Cu at (377.6, 23.7)
- added C18: 22µF, Capacitor_SMD:CP_Elec_6.3x5.8, F.Cu at (377.6, 31.8)
- added C19: 2.2µF, Capacitor_SMD:C_0603_1608Metric_Pad1.08x0.95mm_HandSolder, F.Cu at (373.8, 47.2)
- added C2: 2.2µF, Capacitor_SMD:C_0603_1608Metric_Pad1.08x0.95mm_HandSolder, F.Cu at (369.4, 39.7)
- added C20: 2.2µF, Capacitor_SMD:C_0603_1608Metric_Pad1.08x0.95mm_HandSolder, F.Cu at (373.8, 49.7)
- added C21: DNP, Capacitor_SMD:C_0603_1608Metric_Pad1.08x0.95mm_HandSolder, F.Cu at (373.8, 52.2)
- added C22: DNP, Capacitor_SMD:C_0603_1608Metric_Pad1.08x0.95mm_HandSolder, F.Cu at (373.8, 54.7)
- added C23: 0.1µF, Capacitor_SMD:C_0603_1608Metric_Pad1.08x0.95mm_HandSolder, F.Cu at (378.1, 37.2)
- added C24: 0.1µF, Capacitor_SMD:C_0603_1608Metric_Pad1.08x0.95mm_HandSolder, F.Cu at (378.1, 39.7)
- added C25: 22µF, Capacitor_SMD:CP_Elec_6.3x5.8, F.Cu at (388.1, 15.5)
- added C26: 33µF, Capacitor_SMD:CP_Elec_6.3x5.8, F.Cu at (388.1, 23.7)
- added C27: 33µF, Capacitor_SMD:CP_Elec_6.3x5.8, F.Cu at (388.1, 31.8)
- added C28: 0.1µF, Capacitor_SMD:C_0603_1608Metric_Pad1.08x0.95mm_HandSolder, F.Cu at (415.7, 59.5)
- added C29: 0.1µF, Capacitor_SMD:C_0603_1608Metric_Pad1.08x0.95mm_HandSolder, F.Cu at (415.7, 62.0)
- added C3: DNP, Capacitor_SMD:C_0603_1608Metric_Pad1.08x0.95mm_HandSolder, F.Cu at (369.4, 42.2)
- added C30: 0.1µF, Capacitor_SMD:C_0603_1608Metric_Pad1.08x0.95mm_HandSolder, F.Cu at (415.7, 64.5)
- added C31: 0.1µF, Capacitor_SMD:C_0603_1608Metric_Pad1.08x0.95mm_HandSolder, F.Cu at (415.7, 67.0)
- added C32: 0.1µF, Capacitor_SMD:C_0603_1608Metric_Pad1.08x0.95mm_HandSolder, F.Cu at (415.7, 69.5)
- added C33: 0.1µF, Capacitor_SMD:C_0603_1608Metric_Pad1.08x0.95mm_HandSolder, F.Cu at (415.7, 72.0)
- added C34: 0.1µF, Capacitor_SMD:C_0603_1608Metric_Pad1.08x0.95mm_HandSolder, F.Cu at (415.7, 74.5)
- added C35: 0.1µF, Capacitor_SMD:C_0603_1608Metric_Pad1.08x0.95mm_HandSolder, F.Cu at (420.1, 59.5)
- added C36: 0.1µF, Capacitor_SMD:C_0603_1608Metric_Pad1.08x0.95mm_HandSolder, F.Cu at (420.1, 62.0)
- added C37: 0.1µF, Capacitor_SMD:C_0603_1608Metric_Pad1.08x0.95mm_HandSolder, F.Cu at (420.1, 64.5)
- added C38: 0.1µF, Capacitor_SMD:C_0603_1608Metric_Pad1.08x0.95mm_HandSolder, F.Cu at (420.1, 67.0)
- added C39: 0.1µF, Capacitor_SMD:C_0603_1608Metric_Pad1.08x0.95mm_HandSolder, F.Cu at (420.1, 69.5)
- added C4: DNP, Capacitor_SMD:C_0603_1608Metric_Pad1.08x0.95mm_HandSolder, F.Cu at (369.4, 44.7)
- added C40: 0.1µF, Capacitor_SMD:C_0603_1608Metric_Pad1.08x0.95mm_HandSolder, F.Cu at (420.1, 72.0)
- added C41: 0.1µF, Capacitor_SMD:C_0603_1608Metric_Pad1.08x0.95mm_HandSolder, F.Cu at (420.1, 74.5)
- added C5: 0.1µF, Capacitor_SMD:C_0603_1608Metric_Pad1.08x0.95mm_HandSolder, F.Cu at (369.4, 47.2)
- added C6: 0.1µF, Capacitor_SMD:C_0603_1608Metric_Pad1.08x0.95mm_HandSolder, F.Cu at (369.4, 49.7)
- added C7: 22µF, Capacitor_SMD:CP_Elec_6.3x5.8, F.Cu at (367.2, 15.5)
- added C8: 10µF, Capacitor_SMD:CP_Elec_6.3x5.8, F.Cu at (367.2, 23.7)
- added C9: 22µF, Capacitor_SMD:CP_Elec_6.3x5.8, F.Cu at (367.2, 31.8)
- added D1: LED, LED_SMD:LED_0603_1608Metric_Pad1.05x0.95mm_HandSolder, F.Cu at (425.9, 92.2)
- added D2: LED, LED_SMD:LED_0603_1608Metric_Pad1.05x0.95mm_HandSolder, F.Cu at (433.7, 12.8)
- added D3: LED, LED_SMD:LED_0603_1608Metric_Pad1.05x0.95mm_HandSolder, F.Cu at (433.7, 15.3)
- added D4: LED, LED_SMD:LED_0603_1608Metric_Pad1.05x0.95mm_HandSolder, F.Cu at (433.7, 17.9)
- added D5: LED, LED_SMD:LED_0603_1608Metric_Pad1.05x0.95mm_HandSolder, F.Cu at (433.7, 20.5)
- added D6: LED, LED_SMD:LED_0603_1608Metric_Pad1.05x0.95mm_HandSolder, F.Cu at (433.7, 23.1)
- added D7: LED, LED_SMD:LED_0603_1608Metric_Pad1.05x0.95mm_HandSolder, F.Cu at (433.7, 25.7)
- added D8: LED, LED_SMD:LED_0603_1608Metric_Pad1.05x0.95mm_HandSolder, F.Cu at (433.7, 28.3)
- added J1: 25A Fuse holder, Library:3557-2, F.Cu at (405.8, 52.2)
- added J10: Screw_Terminal_01x02, TerminalBlock_Philmore:TerminalBlock_Philmore_TB132_1x02_P5.00mm_Horizontal, F.Cu at (422.9, 41.8)
- added J11: Conn_01x02, Connector_PinHeader_1.00mm:PinHeader_1x02_P1.00mm_Vertical, F.Cu at (418.0, 49.7)
- added J12: Conn_01x02, Connector_PinHeader_1.00mm:PinHeader_1x02_P1.00mm_Vertical, F.Cu at (25.3, 1.02)
- added J2: Screw_Terminal_01x02, TerminalBlock_Philmore:TerminalBlock_Philmore_TB132_1x02_P5.00mm_Horizontal, F.Cu at (398.8, 17.3)
- added J3: Screw_Terminal_01x02, TerminalBlock_Philmore:TerminalBlock_Philmore_TB132_1x02_P5.00mm_Horizontal, F.Cu at (410.9, 17.3)
- added J4: Screw_Terminal_01x02, TerminalBlock_Philmore:TerminalBlock_Philmore_TB132_1x02_P5.00mm_Horizontal, F.Cu at (422.9, 17.3)
- added J5: Screw_Terminal_01x02, TerminalBlock_Philmore:TerminalBlock_Philmore_TB132_1x02_P5.00mm_Horizontal, F.Cu at (398.8, 29.5)
- added J6: Screw_Terminal_01x02, TerminalBlock_Philmore:TerminalBlock_Philmore_TB132_1x02_P5.00mm_Horizontal, F.Cu at (410.9, 29.5)
- added J7: Screw_Terminal_01x02, TerminalBlock_Philmore:TerminalBlock_Philmore_TB132_1x02_P5.00mm_Horizontal, F.Cu at (422.9, 29.5)
- added J8: Screw_Terminal_01x02, TerminalBlock_Philmore:TerminalBlock_Philmore_TB132_1x02_P5.00mm_Horizontal, F.Cu at (398.8, 41.8)
- added J9: Screw_Terminal_01x02, TerminalBlock_Philmore:TerminalBlock_Philmore_TB132_1x02_P5.00mm_Horizontal, F.Cu at (410.9, 41.8)
- added L1: 33µH, Library:INDPM140128X650N, F.Cu at (353.6, 18.6)
- added L2: 22µH, Library:INDPM140128X650N, F.Cu at (353.6, 33.0)
- added L3: 33µH, Library:INDPM140128X650N, F.Cu at (353.6, 47.3)
- added L4: 22µH, Library:INDPM140128X650N, F.Cu at (353.6, 61.7)
- added L5: 33µH, Library:INDPM140128X650N, F.Cu at (353.6, 76.0)
- added L6: 15µH, Library:INDPM140128X650N, F.Cu at (353.6, 90.4)
- added Q1: LMR51635XDDCR, Library:SOT95P280X110-6N, F.Cu at (364.6, 38.2)
- added Q2: LMR51635XDDCR, Library:SOT95P280X110-6N, F.Cu at (364.6, 42.8)
- added Q3: LMR51635XDDCR, Library:SOT95P280X110-6N, F.Cu at (364.6, 47.4)
- added Q4: LMR51635XDDCR, Library:SOT95P280X110-6N, F.Cu at (364.6, 52.0)
- added Q5: LMR51635XDDCR, Library:SOT95P280X110-6N, F.Cu at (364.6, 56.6)
- added Q6: LMR51635XDDCR, Library:SOT95P280X110-6N, F.Cu at (364.6, 61.2)
- added Q7: BSS84, Package_TO_SOT_SMD:SOT-23, F.Cu at (421.3, 93.3)
- added R1: 10k2, Resistor_SMD:R_0603_1608Metric_Pad0.98x0.95mm_HandSolder, F.Cu at (378.1, 42.2)
- added R10: 10k2, Resistor_SMD:R_0603_1608Metric_Pad0.98x0.95mm_HandSolder, F.Cu at (382.5, 44.7)
- added R11: 194k, Resistor_SMD:R_0603_1608Metric_Pad0.98x0.95mm_HandSolder, F.Cu at (382.5, 47.2)
- added R12: 53k5, Resistor_SMD:R_0603_1608Metric_Pad0.98x0.95mm_HandSolder, F.Cu at (382.5, 49.7)
- added R13: 0.2R, Resistor_SMD:R_Shunt_Vishay_WSK2512_6332Metric_T2.21mm, F.Cu at (408.7, 60.6)
- added R14: 0.2R, Resistor_SMD:R_Shunt_Vishay_WSK2512_6332Metric_T2.21mm, F.Cu at (408.7, 65.5)
- added R15: R50, Resistor_SMD:R_0603_1608Metric_Pad0.98x0.95mm_HandSolder, F.Cu at (424.4, 59.5)
- added R16: R50, Resistor_SMD:R_0603_1608Metric_Pad0.98x0.95mm_HandSolder, F.Cu at (424.4, 62.0)
- added R17: R50, Resistor_SMD:R_0603_1608Metric_Pad0.98x0.95mm_HandSolder, F.Cu at (424.4, 64.5)
- added R18: R50, Resistor_SMD:R_0603_1608Metric_Pad0.98x0.95mm_HandSolder, F.Cu at (424.4, 67.0)
- added R19: 0R, Resistor_SMD:R_0603_1608Metric_Pad0.98x0.95mm_HandSolder, F.Cu at (424.4, 69.5)
- added R2: 10k2, Resistor_SMD:R_0603_1608Metric_Pad0.98x0.95mm_HandSolder, F.Cu at (378.1, 44.7)
- added R20: 1k, Resistor_SMD:R_0603_1608Metric_Pad0.98x0.95mm_HandSolder, F.Cu at (424.4, 72.0)
- added R21: 10k, Resistor_SMD:R_0603_1608Metric_Pad0.98x0.95mm_HandSolder, F.Cu at (424.4, 74.5)
- added R22: 10k, Resistor_SMD:R_0603_1608Metric_Pad0.98x0.95mm_HandSolder, F.Cu at (428.8, 59.5)
- added R23: 330, Resistor_SMD:R_0603_1608Metric_Pad0.98x0.95mm_HandSolder, F.Cu at (428.8, 62.0)
- added R24: 10k, Resistor_SMD:R_0603_1608Metric_Pad0.98x0.95mm_HandSolder, F.Cu at (428.8, 64.5)
- added R25: 10k, Resistor_SMD:R_0603_1608Metric_Pad0.98x0.95mm_HandSolder, F.Cu at (428.8, 67.0)
- added R26: 0.2R, Resistor_SMD:R_Shunt_Vishay_WSK2512_6332Metric_T2.21mm, F.Cu at (408.7, 70.3)
- added R27: 0.2R, Resistor_SMD:R_Shunt_Vishay_WSK2512_6332Metric_T2.21mm, F.Cu at (408.7, 75.2)
- added R28: R50, Resistor_SMD:R_0603_1608Metric_Pad0.98x0.95mm_HandSolder, F.Cu at (428.8, 69.5)
- added R29: R50, Resistor_SMD:R_0603_1608Metric_Pad0.98x0.95mm_HandSolder, F.Cu at (428.8, 72.0)
- added R3: 295k, Resistor_SMD:R_0603_1608Metric_Pad0.98x0.95mm_HandSolder, F.Cu at (378.1, 47.2)
- added R30: R50, Resistor_SMD:R_0603_1608Metric_Pad0.98x0.95mm_HandSolder, F.Cu at (428.8, 74.5)
- added R31: R50, Resistor_SMD:R_0603_1608Metric_Pad0.98x0.95mm_HandSolder, F.Cu at (433.1, 59.5)
- added R32: 10k, Resistor_SMD:R_0603_1608Metric_Pad0.98x0.95mm_HandSolder, F.Cu at (433.1, 62.0)
- added R33: 10k, Resistor_SMD:R_0603_1608Metric_Pad0.98x0.95mm_HandSolder, F.Cu at (433.1, 64.5)
- added R34: 10k, Resistor_SMD:R_0603_1608Metric_Pad0.98x0.95mm_HandSolder, F.Cu at (433.1, 67.0)
- added R35: 10k, Resistor_SMD:R_0603_1608Metric_Pad0.98x0.95mm_HandSolder, F.Cu at (433.1, 69.5)
- added R36: 0.2R, Resistor_SMD:R_Shunt_Vishay_WSK2512_6332Metric_T2.21mm, F.Cu at (408.7, 80.0)
- added R37: 0.2R, Resistor_SMD:R_Shunt_Vishay_WSK2512_6332Metric_T2.21mm, F.Cu at (408.7, 84.9)
- added R38: R50, Resistor_SMD:R_0603_1608Metric_Pad0.98x0.95mm_HandSolder, F.Cu at (433.1, 72.0)
- added R39: R50, Resistor_SMD:R_0603_1608Metric_Pad0.98x0.95mm_HandSolder, F.Cu at (433.1, 74.5)
- added R4: 143k, Resistor_SMD:R_0603_1608Metric_Pad0.98x0.95mm_HandSolder, F.Cu at (378.1, 49.7)
- added R40: R50, Resistor_SMD:R_0603_1608Metric_Pad0.98x0.95mm_HandSolder, F.Cu at (437.5, 59.5)
- added R41: R50, Resistor_SMD:R_0603_1608Metric_Pad0.98x0.95mm_HandSolder, F.Cu at (437.5, 62.0)
- added R42: 10k, Resistor_SMD:R_0603_1608Metric_Pad0.98x0.95mm_HandSolder, F.Cu at (437.5, 64.5)
- added R43: 10k, Resistor_SMD:R_0603_1608Metric_Pad0.98x0.95mm_HandSolder, F.Cu at (437.5, 67.0)
- added R44: 10k, Resistor_SMD:R_0603_1608Metric_Pad0.98x0.95mm_HandSolder, F.Cu at (437.5, 69.5)
- added R45: 10k, Resistor_SMD:R_0603_1608Metric_Pad0.98x0.95mm_HandSolder, F.Cu at (437.5, 72.0)
- added R46: 4k, Resistor_SMD:R_0603_1608Metric_Pad0.98x0.95mm_HandSolder, F.Cu at (433.6, 30.9)
- added R47: 2.2k, Resistor_SMD:R_0603_1608Metric_Pad0.98x0.95mm_HandSolder, F.Cu at (433.6, 33.4)
- added R48: 1.8k, Resistor_SMD:R_0603_1608Metric_Pad0.98x0.95mm_HandSolder, F.Cu at (433.6, 35.9)
- added R49: 1.4k, Resistor_SMD:R_0603_1608Metric_Pad0.98x0.95mm_HandSolder, F.Cu at (433.6, 38.4)
- added R5: 10k2, Resistor_SMD:R_0603_1608Metric_Pad0.98x0.95mm_HandSolder, F.Cu at (378.1, 52.2)
- added R50: 1k, Resistor_SMD:R_0603_1608Metric_Pad0.98x0.95mm_HandSolder, F.Cu at (433.6, 40.9)
- added R51: 330, Resistor_SMD:R_0603_1608Metric_Pad0.98x0.95mm_HandSolder, F.Cu at (433.6, 43.4)
- added R52: 330, Resistor_SMD:R_0603_1608Metric_Pad0.98x0.95mm_HandSolder, F.Cu at (433.6, 45.9)
- added R6: 10k2, Resistor_SMD:R_0603_1608Metric_Pad0.98x0.95mm_HandSolder, F.Cu at (378.1, 54.7)
- added R7: 232k, Resistor_SMD:R_0603_1608Metric_Pad0.98x0.95mm_HandSolder, F.Cu at (382.5, 37.2)
- added R8: 143k, Resistor_SMD:R_0603_1608Metric_Pad0.98x0.95mm_HandSolder, F.Cu at (382.5, 39.7)
- added R9: 10k2, Resistor_SMD:R_0603_1608Metric_Pad0.98x0.95mm_HandSolder, F.Cu at (382.5, 42.2)
- added TP1: TestPoint, TestPoint:TestPoint_Loop_D2.54mm_Drill1.5mm_Beaded, F.Cu at (416.1, 78.3)
- added TP2: TestPoint, TestPoint:TestPoint_Loop_D2.54mm_Drill1.5mm_Beaded, F.Cu at (416.1, 83.3)
- added TP3: TestPoint, TestPoint:TestPoint_Loop_D2.54mm_Drill1.5mm_Beaded, F.Cu at (416.1, 88.4)
- added TP4: TestPoint, TestPoint:TestPoint_Loop_D2.54mm_Drill1.5mm_Beaded, F.Cu at (421.1, 78.3)
- added TP5: TestPoint, TestPoint:TestPoint_Loop_D2.54mm_Drill1.5mm_Beaded, F.Cu at (421.1, 83.3)
- added TP6: TestPoint, TestPoint:TestPoint_Loop_D2.54mm_Drill1.5mm_Beaded, F.Cu at (421.1, 88.4)
- added TP7: TestPoint, TestPoint:TestPoint_Loop_D2.54mm_Drill1.5mm_Beaded, F.Cu at (426.2, 78.3)
- added TP8: TestPoint, TestPoint:TestPoint_Loop_D2.54mm_Drill1.5mm_Beaded, F.Cu at (426.2, 83.3)
- added TP9: TestPoint, TestPoint:TestPoint_Loop_D2.54mm_Drill1.5mm_Beaded, F.Cu at (426.2, 88.4)
- added U1: ACS711xEXLT-31AB, Sensor_Current:Allegro_QFN-12-10-1EP_3x3mm_P0.5mm, F.Cu at (416.2, 93.6)
- added U2: INA219AxD, Package_SO:SOIC-8_3.9x4.9mm_P1.27mm, F.Cu at (399.5, 61.5)
- added U3: INA219AxD, Package_SO:SOIC-8_3.9x4.9mm_P1.27mm, F.Cu at (399.5, 68.1)
- added U4: INA219AxD, Package_SO:SOIC-8_3.9x4.9mm_P1.27mm, F.Cu at (399.5, 74.7)
- added U5: INA219AxD, Package_SO:SOIC-8_3.9x4.9mm_P1.27mm, F.Cu at (399.5, 81.3)
- added U6: INA219AxD, Package_SO:SOIC-8_3.9x4.9mm_P1.27mm, F.Cu at (399.5, 87.9)
- added U7: INA219AxD, Package_SO:SOIC-8_3.9x4.9mm_P1.27mm, F.Cu at (399.5, 94.5)
