File: Hardware/UPD_PCB/UPD_PCB.kicad_sch (KiCad schematic)
At the start: 0 parts

Commit message: Changed text variables
Other:
- note added: "(schematic) connectors"
- note added: "(schematic) current_sensing"
- note added: "(schematic) power_distribution"
- note added: "Schematics"
- note removed: "Random Sheet 1"
- note removed: "Random Sheet 2"
Changed lines of the file:
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@@
 		)
 	)
-	(text "..........................................."
+	(text "(schematic) connectors\n"
 		(exclude_from_sim no)
 		(at 45.72 144.78 0)
@@
 		)
 	)
-	(text "..........................................."
+	(text "(schematic) current_sensing\n"
 		(exclude_from_sim no)
 		(at 45.72 137.16 0)
@@
 		)
 	)
-	(text "Random Sheet 1"
+	(text "Schematics\n"
 		(exclude_from_sim no)
 		(at 45.72 106.68 0)
@@
 		)
 	)
-	(text "Random Sheet 2"
+	(text "Power - Sequencing\n"
 		(exclude_from_sim no)
 		(at 45.72 114.3 0)
@@
 		)
 	)
-	(text "Power - Sequencing"
+	(text "Revision History\n"
 		(exclude_from_sim no)
 		(at 45.72 121.92 0)
@@
 		)
 	)
-	(text "Revision History"
+	(text "(schematic) power_distribution\n"
 		(exclude_from_sim no)
 		(at 45.72 129.54 0)

Commit message: Finalized Schematic
Other:
- title: Cover Page -> Sheet Title A
Changed lines of the file:
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@@
 	(paper "A3")
 	(title_block
-		(title "Cover Page")
+		(title "Sheet Title A")
 		(date "Last Modified Date")
 		(rev "${REVISION}")

Commit message: Updated pcb
Other:
- note added: "Universal power distribution pcb"
- note removed: "Add a comment here"
- note removed: "DESIGN CONSIDERATIONS"
