File: Hardware/UPD_PCB/Project Architecture.kicad_sch (KiCad schematic)
At the start: 0 parts

Commit message: Finalized Schematic
Other:
- title: Project Architecture -> Sheet Title A
Changed lines of the file:
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@@
 	(paper "A3")
 	(title_block
-		(title "Project Architecture")
+		(title "Sheet Title A")
 		(date "Last Modified Date")
 		(rev "${REVISION}")

Commit message: Finalized version V1.0
Changed lines of the file:
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@@
 		)
 	)
-	(text_box "[${#}] ${TITLE}"
+	(text_box "[${#}] Project architecture"
 		(exclude_from_sim no)
 		(at 144.78 20.32 0)
