File: Hardware/UPD_PCB/Section A - Title A.kicad_sch (KiCad schematic)
At the start: 0 parts

Commit message: Finalized version V1.0
Changed lines of the file:
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@@
 		)
 	)
-	(text_box "[${#}] ${TITLE}"
+	(text_box "[${#}] Schematics"
 		(exclude_from_sim no)
 		(at 115.57 15.24 0)
